Commit message: Gazebo plugin for Attitude control of ballbot model
Acceleration is controlled through Attitude references sent to the Gazebo model using this plugin
This simulates the Sliding mode or LQR attitude controller running on the ballbot, ensuring that attitude references are achieved.

File: kugle_description/urdf/gazebo.xacro (robot description, xacro)
@@ -9,6 +9,6 @@
 		<mu1>0.0</mu1>
 		<mu2>0.0</mu2>
-		<kp>1000000.0</kp>
-		<kd>100.0</kd>
+		<!--<kp>1000000.0</kp>
+		<kd>100.0</kd>-->
 		<minDepth>0.001</minDepth>
 		<maxVel>100.0</maxVel>
@@ -24,24 +24,24 @@
 	</gazebo>
 	<gazebo reference="orientation1">
-		<mu1 value="10000.0"/> <!-- Columb friction coefficient in fdir1 direction -->
-		<mu2 value="10000.0"/> <!-- Columb friction in perpendicular direction to fdir1 -->
-		<kp  value="10000000.0" /> <!-- contact stiffness -->
-		<kd  value="1.0" /> <!-- contact damping -->
-		<turnGravityOff>true</turnGravityOff>
+		<mu1 value="0.0"/> <!-- Columb friction coefficient in fdir1 direction -->
+		<mu2 value="0.0"/> <!-- Columb friction in perpendicular direction to fdir1 -->
+		<!--<kp  value="10000000.0" />--> <!-- contact stiffness -->
+		<!--<kd  value="1.0" />--> <!-- contact damping -->
+		<!--<turnGravityOff>true</turnGravityOff>-->
 	</gazebo>
-	<gazebo reference="orientation1">
-		<mu1 value="10000.0"/> <!-- Columb friction coefficient in fdir1 direction -->
-		<mu2 value="10000.0"/> <!-- Columb friction in perpendicular direction to fdir1 -->
-		<kp  value="10000000.0" /> <!-- contact stiffness -->
-		<kd  value="1.0" /> <!-- contact damping -->
-		<turnGravityOff>true</turnGravityOff>
+	<gazebo reference="orientation2">
+		<mu1 value="0.0"/> <!-- Columb friction coefficient in fdir1 direction -->
+		<mu2 value="0.0"/> <!-- Columb friction in perpendicular direction to fdir1 -->
+		<!--<kp  value="10000000.0" />--> <!-- contact stiffness -->
+		<!--<kd  value="1.0" />--> <!-- contact damping -->
+		<!--<turnGravityOff>true</turnGravityOff>-->
 	</gazebo>
 	<gazebo reference="robot">
-		<mu1 value="10000.0"/> <!-- Columb friction coefficient in fdir1 direction -->
-		<mu2 value="10000.0"/> <!-- Columb friction in perpendicular direction to fdir1 -->
-		<kp  value="10000000.0" /> <!-- contact stiffness -->
-		<kd  value="1.0" /> <!-- contact damping -->
+		<mu1 value="0.0"/> <!-- Columb friction coefficient in fdir1 direction -->
+		<mu2 value="0.0"/> <!-- Columb friction in perpendicular direction to fdir1 -->
+		<!--<kp  value="10000000.0" />--> <!-- contact stiffness -->
+		<!--<kd  value="1.0" />--> <!-- contact damping -->
 		<material>Gazebo/Grey</material>
-		<turnGravityOff>true</turnGravityOff>
+		<!--<turnGravityOff>true</turnGravityOff>-->
 	</gazebo>
 	<!-- We need to link Gazebo and ROS and let Gazebo load all the previously defined ROS parameters. Therefore this Gazebo file should be included in the end of the main xacro file! -->
@@ -52,5 +52,5 @@
 		<plugin name="ballbot_acceleration_controller" filename="libgazebo_ballbot_acceleration_control.so">
 			<robotNamespace>/kugle</robotNamespace>
-			<commandTopic>cmd_force</commandTopic>
+			<commandTopic>cmd_attitude</commandTopic>
 			<odometryTopic>odom_raw</odometryTopic>
 			<odometryFrame>odom</odometryFrame>
@@ -59,5 +59,6 @@
 			<robotBaseJoint>base_to_robot</robotBaseJoint>
 			<publishOdometryTf>1</publishOdometryTf>
-			<cmdTimeout>3.0</cmdTimeout>
+			<cmdTimeout>1.0</cmdTimeout>
+			<accelerationCoefficient>13.71</accelerationCoefficient> <!-- Approximate linear relationship between Quaternion reference component and steady state acceleration -->
 		</plugin>
 	</gazebo>

File: kugle_description/urdf/kugle.xacro (robot description, xacro)
@@ -50,11 +50,19 @@
 	<link name="orientation1">
 		<inertial>
-			<xacro:small_inertial/>
+			<origin xyz="0 0 0" rpy="0 0 0" />
+			<mass value="0.001" />
+			<inertia ixx="0.0"
+					 ixy="0"
+					 ixz="0"
+					 iyy="0.0"
+					 iyz="0"
+					 izz="0.0"
+			/>
 		</inertial>
 	</link>
 	<joint name="yaw" type="revolute">
-		<parent link="base_link"/>
+		<parent link="ball"/>
 		<child link="orientation1"/>
-		<origin xyz="0 0 ${ball_radius}" rpy="0 0 0" /> <!-- offset from parent to child, so with direction based in parent frame -->
+		<origin xyz="0 0 0" rpy="0 0 0" /> <!-- offset from parent to child, so with direction based in parent frame -->
 		<axis xyz="0 0 1"/>
 		<limit lower="-${pi}" upper="${pi}" effort="10" velocity="100"/>
@@ -62,5 +70,13 @@
 	<link name="orientation2">
 		<inertial>
-			<xacro:small_inertial/>
+			<origin xyz="0 0 0" rpy="0 0 0" />
+			<mass value="0.001" />
+			<inertia ixx="0.0"
+					 ixy="0"
+					 ixz="0"
+					 iyy="0.0"
+					 iyz="0"
+					 izz="0.0"
+			/>
 		</inertial>
 	</link>
@@ -80,15 +96,15 @@
 			<origin xyz="0 0 ${cylinder_height/2}" rpy="0 0 0" />
 			<mass value="0.001" />
-			<inertia ixx="0.0"
+			<inertia ixx="0000000.0"
 					 ixy="0"
 					 ixz="0"
-					 iyy="0.0"
+					 iyy="0000000.0"
 					 iyz="0"
-					 izz="0.0"
+					 izz="0000000.0"
 			/>
 		</inertial>
-		<collision>
+		<!--<collision>
 			<xacro:robot_geometry/>
-		</collision>
+		</collision>-->
 		<visual>
 			<material name="grey"/>

Commit message: Ballbot attitude control with RVIZ visualization and 3D model
Gazebo simulation model is working and tested
Next step is to add sensors

File: kugle_description/urdf/gazebo.xacro (robot description, xacro)
@@ -23,5 +23,5 @@
 		<!--<turnGravityOff>false</turnGravityOff>-->
 	</gazebo>
-	<gazebo reference="orientation1">
+	<gazebo reference="heading">
 		<mu1 value="0.0"/> <!-- Columb friction coefficient in fdir1 direction -->
 		<mu2 value="0.0"/> <!-- Columb friction in perpendicular direction to fdir1 -->
@@ -30,5 +30,5 @@
 		<!--<turnGravityOff>true</turnGravityOff>-->
 	</gazebo>
-	<gazebo reference="orientation2">
+	<gazebo reference="tilt">
 		<mu1 value="0.0"/> <!-- Columb friction coefficient in fdir1 direction -->
 		<mu2 value="0.0"/> <!-- Columb friction in perpendicular direction to fdir1 -->
@@ -42,5 +42,5 @@
 		<!--<kp  value="10000000.0" />--> <!-- contact stiffness -->
 		<!--<kd  value="1.0" />--> <!-- contact damping -->
-		<material>Gazebo/Grey</material>
+		<!--<material>Gazebo/Grey</material>-->
 		<!--<turnGravityOff>true</turnGravityOff>-->
 	</gazebo>
@@ -52,8 +52,9 @@
 		<plugin name="ballbot_acceleration_controller" filename="libgazebo_ballbot_acceleration_control.so">
 			<robotNamespace>/kugle</robotNamespace>
-			<commandTopic>cmd_attitude</commandTopic>
+			<commandTopic>cmd_quaternion</commandTopic>
 			<odometryTopic>odom_raw</odometryTopic>
 			<odometryFrame>odom</odometryFrame>
 			<odometryRate>20.0</odometryRate>
+			<worldFrame>world</worldFrame>
 			<robotBaseLink>base_link</robotBaseLink>
 			<robotBaseJoint>base_to_robot</robotBaseJoint>

File: kugle_description/urdf/kugle.xacro (robot description, xacro)
@@ -17,5 +17,5 @@
 	<xacro:include filename="$(find kugle_description)/urdf/gazebo.xacro" />
 	<xacro:include filename="$(find kugle_description)/urdf/materials.xacro" />
-	<!-- Base link is center of ball -->
+	<!-- Base link is at the contact point (hence ground level) -->
 	<link name="base_link"/>
 	<!--<link name="contact_point">
@@ -48,5 +48,5 @@
 	</link>
 	<xacro:fixed_offset_joint parent="base_link" child="ball" offset="0 0 ${ball_radius}"/>
-	<link name="orientation1">
+	<link name="heading">
 		<inertial>
 			<origin xyz="0 0 0" rpy="0 0 0" />
@@ -63,10 +63,10 @@
 	<joint name="yaw" type="revolute">
 		<parent link="ball"/>
-		<child link="orientation1"/>
+		<child link="heading"/>
 		<origin xyz="0 0 0" rpy="0 0 0" /> <!-- offset from parent to child, so with direction based in parent frame -->
 		<axis xyz="0 0 1"/>
 		<limit lower="-${pi}" upper="${pi}" effort="10" velocity="100"/>
 	</joint>
-	<link name="orientation2">
+	<link name="tilt">
 		<inertial>
 			<origin xyz="0 0 0" rpy="0 0 0" />
@@ -82,6 +82,6 @@
 	</link>
 	<joint name="pitch" type="revolute">
-		<parent link="orientation1"/>
-		<child link="orientation2"/>
+		<parent link="heading"/>
+		<child link="tilt"/>
 		<origin xyz="0 0 0" rpy="0 0 0" /> <!-- offset from parent to child, so with direction based in parent frame -->
 		<axis xyz="0 1 0"/>
@@ -110,9 +110,13 @@
 			<material name="grey"/>
 			<xacro:robot_geometry/>
+			<!--<origin xyz="0 0 -${ball_radius}" rpy="0 0 ${pi/2}" />
+			<geometry>
+				<mesh filename="package://kugle_gazebo/models/kugle.dae" scale="1.0 1.0 1.0"/>
+			</geometry>-->
 		</visual>
 	</link>
 	<!--<xacro:fixed_offset_joint_rpy parent="base_link" child="robot" offset="0 0 ${ball_radius}" rpy="0.2 0 0" />-->
 	<joint name="roll" type="revolute">
-		<parent link="orientation2"/>
+		<parent link="tilt"/>
 		<child link="robot"/>
 		<origin xyz="0 0 0" rpy="0 0 0" /> <!-- offset from parent to child, so with direction based in parent frame -->

File: kugle_description/urdf/parameters.xacro (robot description, xacro)
@@ -3,5 +3,5 @@
 	<!-- X axis direction is forward, Y axis direction is left -->
 	<!-- Physical properties -->
-	<xacro:property name="ball_radius" value="0.125" />
+	<xacro:property name="ball_radius" value="0.129" />
 	<xacro:property name="ball_mass" value="0.500" />
 	<xacro:property name="cylinder_radius" value="0.100" />

Commit message: Added SICK LiDAR sensors + Realsense RGBD camera

File: kugle_description/urdf/gazebo.xacro (robot description, xacro)
@@ -45,4 +45,14 @@
 		<!--<turnGravityOff>true</turnGravityOff>-->
 	</gazebo>
+	<gazebo reference="sick_left_link">
+		<mu1 value="0.0"/> <!-- Columb friction coefficient in fdir1 direction -->
+		<mu2 value="0.0"/> <!-- Columb friction in perpendicular direction to fdir1 -->
+		<material>Gazebo/Grey</material>
+	</gazebo>
+	<gazebo reference="sick_right_link">
+		<mu1 value="0.0"/> <!-- Columb friction coefficient in fdir1 direction -->
+		<mu2 value="0.0"/> <!-- Columb friction in perpendicular direction to fdir1 -->
+		<material>Gazebo/Grey</material>
+	</gazebo>
 	<!-- We need to link Gazebo and ROS and let Gazebo load all the previously defined ROS parameters. Therefore this Gazebo file should be included in the end of the main xacro file! -->
 	<!-- Link Gazebo and ROS through plugins -->
@@ -67,3 +77,79 @@
 	<!-- hokuyo LiDAR can be found here: https://github.com/mit-racecar/racecar-simulator/blob/master/racecar_description/urdf/racecar.gazebo#L59 -->
 	<!-- camera sensor might be found here: https://github.com/JoshMarino/gazebo_and_ros_control or here: http://gazebosim.org/tutorials?tut=ros_gzplugins -->
+	<gazebo reference="sick_left_link">
+		<!-- SICK TIM571 - https://cdn.sick.com/media/pdf/4/44/444/dataSheet_TiM571-2050101_1075091_en.pdf -->
+		<!-- See also http://wiki.ros.org/sick_tim -->
+		<sensor name="sick_left_sensor" type="ray"> <!-- "ray" or "gpu_ray" -->
+			<pose>0 0 0 0 0 0</pose>
+			<update_rate>15</update_rate>
+			<always_on>${visualize_lidar}</always_on>
+			<visualize>${visualize_lidar}</visualize>
+			<ray>
+				<scan>
+					<horizontal>
+						<samples>810</samples> <!-- 270 deg span with ~0.33 deg (3 scans pr. deg) -->
+						<resolution>1</resolution>
+						<min_angle>-${pi/4}</min_angle> <!-- -45 deg -->
+						<max_angle>${5*pi/4}</max_angle> <!-- 225 deg -->
+					</horizontal>
+				</scan>
+				<range>
+					<min>0.05</min>
+					<max>25.0</max>
+					<resolution>0.01</resolution> <!-- It has not been possible to find this number in the datasheet?! -->
+				</range>
+				<noise>
+					<type>gaussian</type>
+					<!-- Noise parameters based on published spec for SICK TIM571
+                         achieving "+-20mm" accuracy at range < 10m.  A mean of 0.0m and
+                         stddev of 0.02m will put 99.7% of samples within 0.06m of the true
+                         reading. -->
+					<mean>0.0</mean>
+					<stddev>0.02</stddev>
+				</noise>
+			</ray>
+			<plugin name="gazebo_sick_left_controller" filename="libgazebo_ros_laser.so"> <!-- "libgazebo_ros_laser.so" or "libgazebo_ros_gpu_laser.so" -->
+				<topicName>/kugle/laser/left/scan</topicName>
+				<frameName>sick_left_link</frameName>
+			</plugin>
+		</sensor>
+	</gazebo>
+	<gazebo reference="sick_right_link">
+		<!-- SICK TIM571 - https://cdn.sick.com/media/pdf/4/44/444/dataSheet_TiM571-2050101_1075091_en.pdf -->
+		<!-- See also http://wiki.ros.org/sick_tim -->
+		<sensor name="sick_right_sensor" type="ray"> <!-- "ray" or "gpu_ray" -->
+			<pose>0 0 0 0 0 0</pose>
+			<update_rate>15</update_rate>
+			<always_on>${visualize_lidar}</always_on>
+			<visualize>${visualize_lidar}</visualize>
+			<ray>
+				<scan>
+					<horizontal>
+						<samples>810</samples> <!-- 270 deg span with ~0.33 deg (3 scans pr. deg) -->
+						<resolution>1</resolution>
+						<min_angle>-${pi/4}</min_angle> <!-- -45 deg -->
+						<max_angle>${5*pi/4}</max_angle> <!-- 225 deg -->
+					</horizontal>
+				</scan>
+				<range>
+					<min>0.05</min>
+					<max>25.0</max>
+					<resolution>0.01</resolution> <!-- It has not been possible to find this number in the datasheet?! -->
+				</range>
+				<noise>
+					<type>gaussian</type>
+					<!-- Noise parameters based on published spec for SICK TIM571
+                         achieving "+-20mm" accuracy at range < 10m.  A mean of 0.0m and
+                         stddev of 0.02m will put 99.7% of samples within 0.06m of the true
+                         reading. -->
+					<mean>0.0</mean>
+					<stddev>0.02</stddev>
+				</noise>
+			</ray>
+			<plugin name="gazebo_sick_right_controller" filename="libgazebo_ros_laser.so"> <!-- "libgazebo_ros_laser.so" or "libgazebo_ros_gpu_laser.so" -->
+				<topicName>/kugle/laser/right/scan</topicName>
+				<frameName>sick_right_link</frameName>
+			</plugin>
+		</sensor>
+	</gazebo>
 </robot>

File: kugle_description/urdf/kugle.xacro (robot description, xacro)
@@ -61,10 +61,10 @@
 		</inertial>
 	</link>
-	<joint name="yaw" type="revolute">
+	<joint name="yaw" type="continuous">
 		<parent link="ball"/>
 		<child link="heading"/>
 		<origin xyz="0 0 0" rpy="0 0 0" /> <!-- offset from parent to child, so with direction based in parent frame -->
 		<axis xyz="0 0 1"/>
-		<limit lower="-${pi}" upper="${pi}" effort="10" velocity="100"/>
+		<!--<limit lower="-${pi}" upper="${pi}" effort="10" velocity="100"/>-->
 	</joint>
 	<link name="tilt">
@@ -124,3 +124,39 @@
 		<limit lower="-${pi/2}" upper="${pi/2}" effort="10" velocity="100"/>
 	</joint>
+	<link name="sick_left_link">
+		<inertial>
+			<origin xyz="0 0 0" rpy="0 0 0" />
+			<mass value="0.001" />
+			<inertia ixx="0.0"
+					 ixy="0"
+					 ixz="0"
+					 iyy="0.0"
+					 iyz="0"
+					 izz="0.0"
+			/>
+		</inertial>
+		<visual>
+			<material name="grey"/>
+			<xacro:lidar_geometry/>
+		</visual>
+	</link>
+	<xacro:fixed_offset_joint_rpy parent="robot" child="sick_left_link" offset="0 0.123 0.33757" rpy="0 0 0" />
+	<link name="sick_right_link">
+		<inertial>
+			<origin xyz="0 0 0" rpy="0 0 0" />
+			<mass value="0.001" />
+			<inertia ixx="0.0"
+					 ixy="0"
+					 ixz="0"
+					 iyy="0.0"
+					 iyz="0"
+					 izz="0.0"
+			/>
+		</inertial>
+		<visual>
+			<material name="grey"/>
+			<xacro:lidar_geometry/>
+		</visual>
+	</link>
+	<xacro:fixed_offset_joint_rpy parent="robot" child="sick_right_link" offset="0 -0.123 0.33757" rpy="0 0 ${pi}" />
 </robot>

File: kugle_description/urdf/kugle_rviz.xacro (robot description, xacro)
@@ -14,6 +14,4 @@
 	<xacro:include filename="$(find kugle_description)/urdf/joints.xacro" />
 	<xacro:include filename="$(find kugle_description)/urdf/transmissions.xacro" />
-	<!-- Link Gazebo and ROS - this has to happen as the last thing -->
-	<xacro:include filename="$(find kugle_description)/urdf/gazebo.xacro" />
 	<xacro:include filename="$(find kugle_description)/urdf/materials.xacro" />
 	<!-- Base link is at the contact point (hence ground level) -->
@@ -61,10 +59,10 @@
 		</inertial>
 	</link>
-	<joint name="yaw" type="revolute">
+	<joint name="yaw" type="continuous">
 		<parent link="ball"/>
 		<child link="heading"/>
 		<origin xyz="0 0 0" rpy="0 0 0" /> <!-- offset from parent to child, so with direction based in parent frame -->
 		<axis xyz="0 0 1"/>
-		<limit lower="-${pi}" upper="${pi}" effort="10" velocity="100"/>
+		<!--<limit lower="-${pi}" upper="${pi}" effort="10" velocity="100"/>-->
 	</joint>
 	<link name="tilt">
@@ -116,4 +114,5 @@
 		</visual>
 	</link>
+	<!-- Include sensors links -->
 	<!--<xacro:fixed_offset_joint_rpy parent="base_link" child="robot" offset="0 0 ${ball_radius}" rpy="0.2 0 0" />-->
 	<joint name="roll" type="revolute">
@@ -124,3 +123,49 @@
 		<limit lower="-${pi/2}" upper="${pi/2}" effort="10" velocity="100"/>
 	</joint>
+	<link name="sick_left_link">
+		<inertial>
+			<origin xyz="0 0 0" rpy="0 0 0" />
+			<mass value="0.001" />
+			<inertia ixx="0.0"
+					 ixy="0"
+					 ixz="0"
+					 iyy="0.0"
+					 iyz="0"
+					 izz="0.0"
+			/>
+		</inertial>
+		<!--<visual>
+			<material name="grey"/>
+			<xacro:lidar_geometry/>
+		</visual>-->
+	</link>
+	<xacro:fixed_offset_joint_rpy parent="robot" child="sick_left_link" offset="0 0.123 0.33757" rpy="0 0 0" />
+	<link name="sick_right_link">
+		<inertial>
+			<origin xyz="0 0 0" rpy="0 0 0" />
+			<mass value="0.001" />
+			<inertia ixx="0.0"
+					 ixy="0"
+					 ixz="0"
+					 iyy="0.0"
+					 iyz="0"
+					 izz="0.0"
+			/>
+		</inertial>
+		<!--<visual>
+			<material name="grey"/>
+			<xacro:lidar_geometry/>
+		</visual>-->
+	</link>
+	<xacro:fixed_offset_joint_rpy parent="robot" child="sick_right_link" offset="0 -0.123 0.33757" rpy="0 0 ${pi}" />
+	<!-- Link Gazebo and ROS - this has to happen as the last thing -->
+	<xacro:include filename="$(find kugle_description)/urdf/gazebo.xacro" />
+	<!-- Add realsense camera link -->
+	<!-- Note that this Realsense camera is not the correct one, hence the physical location (frames) of the different image streams will be different in real life -->
+	<!-- Import macro for realsense-RS200 camera-->
+	<xacro:include filename="$(find realsense_gazebo_plugin)/urdf/realsense-RS200.macro.xacro"/>
+	<!-- Create camera instance -->
+	<xacro:realsense-rs200 prefix="" parent="robot">
+		<origin xyz="0.05 0 1.11" rpy="0 0.25 0" />
+	</xacro:realsense-rs200>
 </robot>

File: kugle_description/urdf/parameters.xacro (robot description, xacro)
@@ -6,5 +6,7 @@
 	<xacro:property name="ball_mass" value="0.500" />
 	<xacro:property name="cylinder_radius" value="0.100" />
-	<xacro:property name="cylinder_height" value="0.500" />
+	<xacro:property name="cylinder_height" value="1.000" />
 	<xacro:property name="cylinder_mass" value="0.500" />
+	<!-- Sensor parameters -->
+	<xacro:property name="visualize_lidar" value="false" />
 </robot>

File: kugle_description/urdf/physical.xacro (robot description, xacro)
@@ -31,3 +31,11 @@
 		<xacro:cylinder_inertial mass="${cylinder_mass}" radius="${cylinder_radius}" length="${cylinder_height}" />
 	</xacro:macro>
+	<!-- LiDAR geometry -->
+	<xacro:macro name="lidar_geometry">
+		<origin xyz="0 0 -0.019585" rpy="0 0 0" />
+		<geometry>
+			<!-- SICK TIM571 LiDAR bounding box -->
+			<box size="0.060 0.061 0.08575" />
+		</geometry>
+	</xacro:macro>
 </robot>
